File: PCB/Skeleton68rev2.kicad_pcb (KiCad board)
At the start: 2 copper layers, 180 parts, among them J1 USB_C_Receptacle_USB2.0, SW1 SW_Push, SW10 SW_Push, SW11 SW_Push, SW12 SW_Push, SW13 SW_Push, SW14 SW_Push, SW15 SW_Push, SW16 SW_Push, SW17 SW_Push, SW18 SW_Push, SW19 SW_Push, SW2 SW_Push, SW20 SW_Push, SW21 SW_Push, SW22 SW_Push, SW23 SW_Push, SW24 SW_Push, SW25 SW_Push, SW26 SW_Push, SW27 SW_Push, SW28 SW_Push, SW29 SW_Push, SW3 SW_Push, SW30 SW_Push, SW31 SW_Push, SW32 SW_Push, SW33 SW_Push, SW34 SW_Push, SW35 SW_Push, SW36 SW_Push, SW37 SW_Push, SW38 SW_Push, SW39 SW_Push, SW4 SW_Push, SW40 SW_Push, SW41 SW_Push, SW42 SW_Push, SW43 SW_Push, SW44 SW_Push, SW45 SW_Push, SW46 SW_Push, SW47 SW_Push, SW48 SW_Push, SW49 SW_Push, SW5 SW_Push, SW50 SW_Push, SW51 SW_Push, SW52 SW_Push, SW53 SW_Push, SW54 SW_Push, SW55 SW_Push, SW56 SW_Push, SW57 SW_Push, SW58 SW_Push, SW59 SW_Push, SW6 SW_Push, SW60 SW_Push, SW61 SW_Push, SW62 SW_Push, SW63 SW_Push, SW64 SW_Push, SW65 SW_Push, SW66 SW_Push, SW67 SW_Push, SW68 SW_Push, SW7 SW_Push, SW8 SW_Push, SW9 SW_Push, U1 W25Q128JVS, U2 USBLC6-2SC6, U3 RP2040, U4 XC6206PxxxMR, Y1 12MHz

Commit message: ライセンス変更
Parts:
- J1: moved to B.Cu
- moved SW15 607.7 mm to (344.5, 33.4)
- moved SW14 572.0 mm to (307.9, 35.6)
- moved SW12 567.5 mm to (260.2, 34.9)
- moved J1 490.6 mm to (169.0, 20.8)
- moved SW10 464.0 mm to (220.8, 40.4), turned to 12 degrees
- moved SW9 406.2 mm to (202.1, 44.4), turned to 12 degrees
- moved SW6 401.1 mm to (136.6, 46.4), turned to -12 degrees
- moved SW13 380.7 mm to (279.3, 35.6)
- moved SW11 341.3 mm to (239.4, 36.5), turned to 12 degrees
- moved SW1 327.1 mm to (40.8, 35.6)
- moved SW8 325.6 mm to (183.5, 48.4), turned to 12 degrees
- moved SW4 322.7 mm to (99.3, 38.5), turned to -12 degrees
- moved SW2 295.1 mm to (59.9, 35.6)
- moved SW5 283.2 mm to (117.9, 42.4), turned to -12 degrees
- moved SW7 261.6 mm to (155.2, 50.3), turned to -12 degrees
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Other:
- board outline added: 631.4 x 140.9 mm
