File: PCB/Skeleton68rev2.kicad_sch (KiCad schematic)
At the start: 180 parts, among them J1 USB_C_Receptacle_USB2.0, SW1 SW_Push, SW10 SW_Push, SW11 SW_Push, SW12 SW_Push, SW13 SW_Push, SW14 SW_Push, SW15 SW_Push, SW16 SW_Push, SW17 SW_Push, SW18 SW_Push, SW19 SW_Push, SW2 SW_Push, SW20 SW_Push, SW21 SW_Push, SW22 SW_Push, SW23 SW_Push, SW24 SW_Push, SW25 SW_Push, SW26 SW_Push, SW27 SW_Push, SW28 SW_Push, SW29 SW_Push, SW3 SW_Push, SW30 SW_Push, SW31 SW_Push, SW32 SW_Push, SW33 SW_Push, SW34 SW_Push, SW35 SW_Push, SW36 SW_Push, SW37 SW_Push, SW38 SW_Push, SW39 SW_Push, SW4 SW_Push, SW40 SW_Push, SW41 SW_Push, SW42 SW_Push, SW43 SW_Push, SW44 SW_Push, SW45 SW_Push, SW46 SW_Push, SW47 SW_Push, SW48 SW_Push, SW49 SW_Push, SW5 SW_Push, SW50 SW_Push, SW51 SW_Push, SW52 SW_Push, SW53 SW_Push, SW54 SW_Push, SW55 SW_Push, SW56 SW_Push, SW57 SW_Push, SW58 SW_Push, SW59 SW_Push, SW6 SW_Push, SW60 SW_Push, SW61 SW_Push, SW62 SW_Push, SW63 SW_Push, SW64 SW_Push, SW65 SW_Push, SW66 SW_Push, SW67 SW_Push, SW68 SW_Push, SW7 SW_Push, SW8 SW_Push, SW9 SW_Push, U1 W25Q128JVS, U2 USBLC6-2SC6, U3 RP2040, U4 XC6206PxxxMR, Y1 12MHz

Commit message: 仮配線
Parts:
- SW1, SW10, SW11, SW12, SW13, SW15, SW17, SW18, SW19, SW2, SW20, SW21, SW22, SW23, SW24, SW25, SW26, SW27, SW28, SW3, SW30, SW32, SW33, SW34, SW35, SW36, SW37, SW38, SW39, SW4, SW40, SW41, SW42, SW44, SW46, SW47, SW48, SW49, SW5, SW50, SW51, SW52, SW53, SW54, SW55, SW56, SW58, SW6, SW62, SW66, SW67, SW68, SW7, SW8, SW9: footprint MX_Hotswap:MX-Hotswap-1U -> CustomKey:MX-Hotswap-1U
- SW14: footprint MX_Hotswap:MX-Hotswap-1U -> CustomKey:MX-Hotswap-2U
- SW16, SW29, SW59, SW60, SW64, SW65: footprint MX_Hotswap:MX-Hotswap-1U -> CustomKey:MX-Hotswap-1.5U
- SW31, SW57: footprint MX_Hotswap:MX-Hotswap-1U -> CustomKey:MX-Hotswap-1.75U
- SW43, SW45: footprint MX_Hotswap:MX-Hotswap-1U -> CustomKey:MX-Hotswap-2.25U
- SW61: footprint MX_Hotswap:MX-Hotswap-1U -> CustomKey:MX-Hotswap-2.25U-ReversedStabilizers
- SW63: footprint MX_Hotswap:MX-Hotswap-1U -> CustomKey:MX-Hotswap-2.75U-ReversedStabilizers
Connections:
- net col0: now also U3.32 (GPIO21); no longer U3.7 (GPIO5)
- net col1: now also U3.34 (GPIO22); no longer U3.8 (GPIO6)
- net col10: now also U3.8 (GPIO6); no longer U3.18 (GPIO15)
- net col11: now also U3.12 (GPIO9); no longer U3.27 (GPIO16)
- net col12: now also U3.13 (GPIO10); no longer U3.28 (GPIO17)
- net col13: now also U3.14 (GPIO11); no longer U3.29 (GPIO18)
- net col14: now also U3.15 (GPIO12); no longer U3.30 (GPIO19)
- net col15: now also U3.16 (GPIO13); no longer U3.31 (GPIO20)
- net col2: now also U3.35 (GPIO23); no longer U3.9 (GPIO7)
- net col3: now also U3.36 (GPIO24); no longer U3.11 (GPIO8)
- net col4: now also U3.37 (GPIO25); no longer U3.12 (GPIO9)
- net col5: now also U3.38 (GPIO26_ADC0); no longer U3.13 (GPIO10)
- net col6: now also U3.39 (GPIO27_ADC1); no longer U3.14 (GPIO11)
- net col7: now also U3.5 (GPIO3); no longer U3.15 (GPIO12)
- net col8: now also U3.6 (GPIO4); no longer U3.16 (GPIO13)
- net col9: now also U3.7 (GPIO5); no longer U3.17 (GPIO14)
- net row0: now also U3.41 (GPIO29_ADC3); no longer U3.2 (GPIO0)
- net row1: now also U3.40 (GPIO28_ADC2); no longer U3.3 (GPIO1)
- net row2: now also U3.31 (GPIO20); no longer U3.4 (GPIO2)
- net row3: now also U3.30 (GPIO19); no longer U3.5 (GPIO3)
- net row4: now also U3.29 (GPIO18); no longer U3.6 (GPIO4)
- net underglow: no longer U3.37 (GPIO25)
- no-connect marks 13 -> 14

Commit message: side mounted LEDs
Parts:
- added FID1, FID2, FID3, FID4: Fiducial, Fiducial:Fiducial_1mm_Mask2mm, symbol Mechanical:Fiducial
- added H7, H8: MountingHole, MountingHole:MountingHole_2.2mm_M2, symbol Mechanical:MountingHole
- added LED10, LED11, LED12, LED13, LED14, LED15, LED16, LED17, LED18, LED19, LED20, LED21, LED22, LED23, LED24, LED25, LED26, LED27, LED28, LED29, LED30, LED31, LED6, LED7, LED8, LED9: WS2812B-4020, SkeletonKBD:WS2812B-4020, symbol SkeletonKBD:WS2812B-4020
- D1, D10, D11, D12, D13, D14, D15, D16, D17, D18, D19, D2, D20, D21, D22, D23, D24, D25, D26, D27, D28, D29, D3, D30, D31, D32, D33, D34, D35, D36, D37, D38, D39, D4, D40, D41, D42, D43, D44, D45, D46, D47, D48, D49, D5, D50, D51, D52, D53, D54, D55, D56, D57, D58, D59, D6, D60, D61, D62, D63, D64, D65, D66, D67, D68, D7, D8, D9: LCSC (none) -> C81598; MPN (none) -> 1N4148W
- LED1, LED2, LED3, LED4, LED5: LCSC (none) -> C965557
- SW1, SW10, SW11, SW12, SW13, SW14, SW15, SW16, SW17, SW18, SW19, SW2, SW20, SW21, SW22, SW23, SW24, SW25, SW26, SW27, SW28, SW29, SW3, SW30, SW31, SW32, SW33, SW34, SW35, SW36, SW37, SW38, SW39, SW4, SW40, SW41, SW42, SW43, SW44, SW45, SW46, SW47, SW48, SW49, SW5, SW50, SW51, SW52, SW53, SW54, SW55, SW56, SW57, SW58, SW59, SW6, SW60, SW61, SW62, SW63, SW64, SW65, SW66, SW67, SW68, SW7, SW8, SW9: LCSC (none) -> C2803348
- U3: LCSC (none) -> C2040
Connections:
- net +5V: now also LED10.2 (VDD), LED11.2 (VDD), LED12.2 (VDD), LED13.2 (VDD), LED14.2 (VDD), LED15.2 (VDD), LED16.2 (VDD), LED17.2 (VDD), LED18.2 (VDD), LED19.2 (VDD), LED20.2 (VDD), LED21.2 (VDD), LED22.2 (VDD), LED23.2 (VDD), LED24.2 (VDD), LED25.2 (VDD), LED26.2 (VDD), LED27.2 (VDD), LED28.2 (VDD), LED29.2 (VDD), LED30.2 (VDD), LED31.2 (VDD), LED6.2 (VDD), LED7.2 (VDD), LED8.2 (VDD), LED9.2 (VDD)
- net GND: now also LED10.4 (VSS), LED11.4 (VSS), LED12.4 (VSS), LED13.4 (VSS), LED14.4 (VSS), LED15.4 (VSS), LED16.4 (VSS), LED17.4 (VSS), LED18.4 (VSS), LED19.4 (VSS), LED20.4 (VSS), LED21.4 (VSS), LED22.4 (VSS), LED23.4 (VSS), LED24.4 (VSS), LED25.4 (VSS), LED26.4 (VSS), LED27.4 (VSS), LED28.4 (VSS), LED29.4 (VSS), LED30.4 (VSS), LED31.4 (VSS), LED6.4 (VSS), LED7.4 (VSS), LED8.4 (VSS), LED9.4 (VSS)
- net underglow: now also U3.2 (GPIO0)
- net at LED5.3 (DOUT): now also LED6.1 (DIN)
- new net: LED14.3 (DOUT), LED15.1 (DIN)
- new net: LED15.3 (DOUT), LED16.1 (DIN)
- new net: LED11.3 (DOUT), LED12.1 (DIN)
- new net: LED12.3 (DOUT), LED13.1 (DIN)
- new net: LED29.3 (DOUT), LED30.1 (DIN)
- new net: LED30.3 (DOUT), LED31.1 (DIN)
- new net: LED16.3 (DOUT), LED17.1 (DIN)
- new net: LED17.3 (DOUT), LED18.1 (DIN)
- new net: LED18.3 (DOUT), LED19.1 (DIN)
- new net: LED25.3 (DOUT), LED26.1 (DIN)
- new net: LED26.3 (DOUT), LED27.1 (DIN)
- new net: LED6.3 (DOUT), LED7.1 (DIN)
- new net: LED7.3 (DOUT), LED8.1 (DIN)
- new net: LED23.3 (DOUT), LED24.1 (DIN)
- new net: LED24.3 (DOUT), LED25.1 (DIN)
- new net: LED19.3 (DOUT), LED20.1 (DIN)
- new net: LED20.3 (DOUT), LED21.1 (DIN)
- new net: LED13.3 (DOUT), LED14.1 (DIN)
- new net: LED8.3 (DOUT), LED9.1 (DIN)
- new net: LED10.1 (DIN), LED9.3 (DOUT)
- new net: LED10.3 (DOUT), LED11.1 (DIN)
- new net: LED21.3 (DOUT), LED22.1 (DIN)
- new net: LED22.3 (DOUT), LED23.1 (DIN)
- new net: LED27.3 (DOUT), LED28.1 (DIN)
- new net: LED28.3 (DOUT), LED29.1 (DIN)
- no-connect marks 14 -> 13

Commit message: v1.0
Parts:
- removed LED1, LED10, LED11, LED12, LED13, LED14, LED15, LED16, LED17, LED18, LED19, LED2, LED20, LED21, LED22, LED23, LED24, LED25, LED26, LED27, LED28, LED29, LED3, LED30, LED31, LED4, LED5, LED6, LED7, LED8, LED9: WS2812B-4020, SkeletonKBD:WS2812B-4020, symbol SkeletonKBD:WS2812B-4020
- added LED1, LED10, LED11, LED12, LED13, LED14, LED15, LED16, LED17, LED18, LED19, LED2, LED20, LED21, LED22, LED23, LED24, LED25, LED26, LED27, LED28, LED29, LED3, LED30, LED31, LED32, LED33, LED34, LED35, LED36, LED37, LED38, LED39, LED4, LED40, LED41, LED42, LED43, LED44, LED45, LED46, LED47, LED48, LED49, LED5, LED50, LED51, LED52, LED53, LED54, LED55, LED56, LED57, LED58, LED59, LED6, LED60, LED61, LED62, LED63, LED64, LED65, LED66, LED67, LED68, LED7, LED8, LED9: SK6812mini-e, Keebio-Parts:SK6812-MINI-E, symbol LED:WS2812B
- added Q1: BSS138, Package_TO_SOT_SMD:SOT-23, symbol Transistor_FET:BSS138
- added R8, R9: 10k, Resistor_SMD:R_0603_1608Metric, symbol Device:R_Small
- H1, H2, H3, H4, H5, H6, H7, H8: footprint MountingHole:MountingHole_2.2mm_M2 -> MountingHole:MountingHole_2.2mm_M2_Pad_Via
- R5, R6: value 27R -> 27
- SW1, SW10, SW11, SW12, SW13, SW14, SW15, SW16, SW17, SW18, SW19, SW2, SW20, SW21, SW22, SW23, SW24, SW25, SW26, SW27, SW28, SW29, SW3, SW30, SW31, SW32, SW33, SW34, SW35, SW36, SW37, SW38, SW39, SW4, SW40, SW41, SW42, SW43, SW44, SW45, SW46, SW47, SW48, SW49, SW5, SW50, SW51, SW52, SW53, SW54, SW55, SW56, SW57, SW58, SW59, SW6, SW60, SW61, SW62, SW63, SW64, SW65, SW66, SW67, SW68, SW7, SW8, SW9: MPN (none) -> CPG151101S11
- TS1, TS2: LCSC C318884 -> C318884
- U3: MPN (none) -> RP2040
Connections:
- net +3V3: now also Q1.1 (G), R8.1
- net +5V: now also LED1.1 (VDD), LED10.1 (VDD), LED11.1 (VDD), LED12.1 (VDD), LED13.1 (VDD), LED14.1 (VDD), LED15.1 (VDD), LED16.1 (VDD), LED17.1 (VDD), LED18.1 (VDD), LED19.1 (VDD), LED2.1 (VDD), LED20.1 (VDD), LED21.1 (VDD), LED22.1 (VDD), LED23.1 (VDD), LED24.1 (VDD), LED25.1 (VDD), LED26.1 (VDD), LED27.1 (VDD), LED28.1 (VDD), LED29.1 (VDD), LED3.1 (VDD), LED30.1 (VDD), LED31.1 (VDD), LED32.1 (VDD), LED33.1 (VDD), LED34.1 (VDD), LED35.1 (VDD), LED36.1 (VDD), LED37.1 (VDD), LED38.1 (VDD), LED39.1 (VDD), LED4.1 (VDD), LED40.1 (VDD), LED41.1 (VDD), LED42.1 (VDD), LED43.1 (VDD), LED44.1 (VDD), LED45.1 (VDD), LED46.1 (VDD), LED47.1 (VDD), LED48.1 (VDD), LED49.1 (VDD), LED5.1 (VDD), LED50.1 (VDD), LED51.1 (VDD), LED52.1 (VDD), LED53.1 (VDD), LED54.1 (VDD), LED55.1 (VDD), LED56.1 (VDD), LED57.1 (VDD), LED58.1 (VDD), LED59.1 (VDD), LED6.1 (VDD), LED60.1 (VDD), LED61.1 (VDD), LED62.1 (VDD), LED63.1 (VDD), LED64.1 (VDD), LED65.1 (VDD), LED66.1 (VDD), LED67.1 (VDD), LED68.1 (VDD), LED7.1 (VDD), LED8.1 (VDD), LED9.1 (VDD), R9.1
- net GND: now also LED1.3 (VSS), LED10.3 (VSS), LED11.3 (VSS), LED12.3 (VSS), LED13.3 (VSS), LED14.3 (VSS), LED15.3 (VSS), LED16.3 (VSS), LED17.3 (VSS), LED18.3 (VSS), LED19.3 (VSS), LED2.3 (VSS), LED20.3 (VSS), LED21.3 (VSS), LED22.3 (VSS), LED23.3 (VSS), LED24.3 (VSS), LED25.3 (VSS), LED26.3 (VSS), LED27.3 (VSS), LED28.3 (VSS), LED29.3 (VSS), LED3.3 (VSS), LED30.3 (VSS), LED31.3 (VSS), LED32.3 (VSS), LED33.3 (VSS), LED34.3 (VSS), LED35.3 (VSS), LED36.3 (VSS), LED37.3 (VSS), LED38.3 (VSS), LED39.3 (VSS), LED4.3 (VSS), LED40.3 (VSS), LED41.3 (VSS), LED42.3 (VSS), LED43.3 (VSS), LED44.3 (VSS), LED45.3 (VSS), LED46.3 (VSS), LED47.3 (VSS), LED48.3 (VSS), LED49.3 (VSS), LED5.3 (VSS), LED50.3 (VSS), LED51.3 (VSS), LED52.3 (VSS), LED53.3 (VSS), LED54.3 (VSS), LED55.3 (VSS), LED56.3 (VSS), LED57.3 (VSS), LED58.3 (VSS), LED59.3 (VSS), LED6.3 (VSS), LED60.3 (VSS), LED61.3 (VSS), LED62.3 (VSS), LED63.3 (VSS), LED64.3 (VSS), LED65.3 (VSS), LED66.3 (VSS), LED67.3 (VSS), LED68.3 (VSS), LED7.3 (VSS), LED8.3 (VSS), LED9.3 (VSS)
- net col6: now also U3.40 (GPIO28_ADC2); no longer U3.39 (GPIO27_ADC1)
- net row1: now also U3.39 (GPIO27_ADC1); no longer U3.40 (GPIO28_ADC2)
- net underglow renamed rgb
- net rgb: now also Q1.2 (S), R8.2
- new net: LED19.2 (DOUT), LED20.4 (DIN)
- new net: LED18.2 (DOUT), LED19.4 (DIN)
- new net: LED52.2 (DOUT), LED53.4 (DIN)
- new net: LED51.2 (DOUT), LED52.4 (DIN)
- new net: LED31.2 (DOUT), LED32.4 (DIN)
- new net: LED30.2 (DOUT), LED31.4 (DIN)
- new net: LED10.2 (DOUT), LED11.4 (DIN)
- new net: LED10.4 (DIN), LED9.2 (DOUT)
- new net: LED36.2 (DOUT), LED37.4 (DIN)
- new net: LED35.2 (DOUT), LED36.4 (DIN)
- new net: LED60.2 (DOUT), LED61.4 (DIN)
- new net: LED59.2 (DOUT), LED60.4 (DIN)
- new net: LED14.2 (DOUT), LED15.4 (DIN)
- new net: LED13.2 (DOUT), LED14.4 (DIN)
- new net: LED1.2 (DOUT), LED2.4 (DIN)
- new net: LED39.2 (DOUT), LED40.4 (DIN)
- new net: LED38.2 (DOUT), LED39.4 (DIN)
- new net: LED61.2 (DOUT), LED62.4 (DIN)
- new net: LED29.2 (DOUT), LED30.4 (DIN)
- new net: LED50.2 (DOUT), LED51.4 (DIN)
- new net: LED49.2 (DOUT), LED50.4 (DIN)
- new net: LED22.2 (DOUT), LED23.4 (DIN)
- new net: LED21.2 (DOUT), LED22.4 (DIN)
- new net: LED58.2 (DOUT), LED59.4 (DIN)
- new net: LED57.2 (DOUT), LED58.4 (DIN)
- new net: LED41.2 (DOUT), LED42.4 (DIN)
- new net: LED40.2 (DOUT), LED41.4 (DIN)
- new net: LED3.2 (DOUT), LED4.4 (DIN)
- new net: LED2.2 (DOUT), LED3.4 (DIN)
- new net: LED67.2 (DOUT), LED68.4 (DIN)
- new net: LED66.2 (DOUT), LED67.4 (DIN)
- new net: LED8.2 (DOUT), LED9.4 (DIN)
- new net: LED16.2 (DOUT), LED17.4 (DIN)
- new net: LED15.2 (DOUT), LED16.4 (DIN)
- new net: LED46.2 (DOUT), LED47.4 (DIN)
- new net: LED45.2 (DOUT), LED46.4 (DIN)
- new net: LED65.2 (DOUT), LED66.4 (DIN)
- new net: LED4.2 (DOUT), LED5.4 (DIN)
- new net: LED28.2 (DOUT), LED29.4 (DIN)
- new net: LED27.2 (DOUT), LED28.4 (DIN)
- new net: LED26.2 (DOUT), LED27.4 (DIN)
- new net: LED25.2 (DOUT), LED26.4 (DIN)
- new net: LED56.2 (DOUT), LED57.4 (DIN)
- new net: LED55.2 (DOUT), LED56.4 (DIN)
- new net: LED48.2 (DOUT), LED49.4 (DIN)
- new net: LED47.2 (DOUT), LED48.4 (DIN)
- new net: LED54.2 (DOUT), LED55.4 (DIN)
- new net: LED53.2 (DOUT), LED54.4 (DIN)
- new net: LED24.2 (DOUT), LED25.4 (DIN)
- new net: LED23.2 (DOUT), LED24.4 (DIN)
- new net: LED20.2 (DOUT), LED21.4 (DIN)
- new net: LED64.2 (DOUT), LED65.4 (DIN)
- new net: LED63.2 (DOUT), LED64.4 (DIN)
- new net: LED12.2 (DOUT), LED13.4 (DIN)
- new net: LED11.2 (DOUT), LED12.4 (DIN)
- new net: LED34.2 (DOUT), LED35.4 (DIN)
- new net: LED33.2 (DOUT), LED34.4 (DIN)
- new net: LED42.2 (DOUT), LED43.4 (DIN)
- new net: LED7.2 (DOUT), LED8.4 (DIN)
- new net: LED17.2 (DOUT), LED18.4 (DIN)
- new net: LED5.2 (DOUT), LED6.4 (DIN)
- new net: LED44.2 (DOUT), LED45.4 (DIN)
- new net: LED43.2 (DOUT), LED44.4 (DIN)
- new net: LED62.2 (DOUT), LED63.4 (DIN)
- new net: LED32.2 (DOUT), LED33.4 (DIN)
- new net: LED6.2 (DOUT), LED7.4 (DIN)
- new net: LED37.2 (DOUT), LED38.4 (DIN)
- new net led: LED1.4 (DIN), Q1.3 (D), R9.2

Commit message: extend sk6812mini-e holes
Parts:
- LED1, LED10, LED11, LED12, LED13, LED14, LED15, LED16, LED17, LED18, LED19, LED2, LED20, LED21, LED22, LED23, LED24, LED25, LED26, LED27, LED28, LED29, LED3, LED30, LED31, LED32, LED33, LED34, LED35, LED36, LED37, LED38, LED39, LED4, LED40, LED41, LED42, LED43, LED44, LED45, LED46, LED47, LED48, LED49, LED5, LED50, LED51, LED52, LED53, LED54, LED55, LED56, LED57, LED58, LED59, LED6, LED60, LED61, LED62, LED63, LED64, LED65, LED66, LED67, LED68, LED7, LED8, LED9: footprint Keebio-Parts:SK6812-MINI-E -> CustomKey:SK6812-MINI-E
