File: SwitchPlate/Skeleton68rev2_SwitchPlate.kicad_pcb (KiCad board)
At the start: 2 copper layers, 349.7 x 118 mm, 0 parts

Commit message: Add Plate
Other:
- board size 349.7 x 118 mm -> 350 x 120.2 mm
- board text added: "V-Cut->"
- board text removed: "<- V-Cut"
- board text removed: "V-Cut ->"

Commit message: extend sk6812mini-e holes
Parts:
- added REF**: mousebite, mousebites:mousebite, F.Cu at (300.0, 91.0)
- added REF**: mousebite, mousebites:mousebite, F.Cu at (300.0, 11.0)
- added REF**: mousebite, mousebites:mousebite, F.Cu at (312.5, 11.0)
- added REF**: mousebite, mousebites:mousebite, F.Cu at (295.8, 11.0)
Other:
- board size 350 x 120.2 mm -> 336.8 x 113.2 mm
- board text removed: "V-Cut->"
